File: Anti-Spark-Switch.sch (KiCad schematic (older format))
At the start: 9 parts

Commit message: schematic completed, PCB started
Parts:
- removed Q? (x3): IRFS7530, sparkparts:D2PAK-7-GDS, symbol IRFS7530
- added P1, P2, P5, P6: Pad_Conn, sparkparts:1PAD_6x5mm, symbol Pad_Conn
- added P3, P4: Screw_Terminal, sparkparts:M5_Screw_Terminal_12_pin, symbol Screw_Terminal
- added P7: CONN_01X02, Connect:PINHEAD1-2, symbol CONN_01X02
- added Q1, Q2, Q3: IRFS7530, sparkparts:D2PAK-7-GDS, symbol IRFS7530
- C1: renamed from C?; footprint (none) -> Capacitors_SMD:C_0603
- D1: renamed from D?; footprint (none) -> Diodes_SMD:SOD-123
- R1, R2, R3: renamed from R?; footprint (none) -> Resistors_SMD:R_0603
- SW1: renamed from SW?; footprint (none) -> Connect:PINHEAD1-3
Connections:
- net labels added: +12V
- wire segments 41 -> 28
Other:
- note added: "12V supplied externally"
- note added: "12V supply for optional LED button"
- note added: "Fuse holder, 30mm spacing between screw terminals\n"
Changed lines of the file:
@@
 LIBS:valves
 LIBS:sparkparts
+LIBS:crf_1
 LIBS:Anti-Spark-Switch-cache
 EELAYER 25 0
@@
 $EndDescr
 $Comp
-L R R?
+L R R2
 U 1 1 5775E315
 P 3100 3800
-F 0 "R?" V 3180 3800 50  0000 C CNN
+F 0 "R2" V 3180 3800 50  0000 C CNN
 F 1 "1M" V 3100 3800 50  0000 C CNN
-F 2 "" V 3030 3800 50  0000 C CNN
+F 2 "Resistors_SMD:R_0603" V 3030 3800 50  0001 C CNN
 F 3 "" H 3100 3800 50  0000 C CNN
 	1    3100 3800
@@
 $EndComp
 $Comp
-L R R?
+L R R1
 U 1 1 5775E3D7
 P 3100 3200
-F 0 "R?" V 3180 3200 50  0000 C CNN
+F 0 "R1" V 3180 3200 50  0000 C CNN
 F 1 "1M" V 3100 3200 50  0000 C CNN
-F 2 "" V 3030 3200 50  0000 C CNN
+F 2 "Resistors_SMD:R_0603" V 3030 3200 50  0001 C CNN
 F 3 "" H 3100 3200 50  0000 C CNN
 	1    3100 3200
@@
 $EndComp
 $Comp
-L R R?
+L R R3
 U 1 1 5775E416
 P 3800 3100
-F 0 "R?" V 3880 3100 50  0000 C CNN
+F 0 "R3" V 3880 3100 50  0000 C CNN
 F 1 "1K" V 3800 3100 50  0000 C CNN
-F 2 "" V 3730 3100 50  0000 C CNN
+F 2 "Resistors_SMD:R_0603" V 3730 3100 50  0001 C CNN
 F 3 "" H 3800 3100 50  0000 C CNN
 	1    3800 3100
@@
 $EndComp
 $Comp
-L C C?
+L C C1
 U 1 1 5775E442
 P 3500 3300
-F 0 "C?" H 3525 3400 50  0000 L CNN
+F 0 "C1" H 3525 3400 50  0000 L CNN
 F 1 "1uF" H 3525 3200 50  0000 L CNN
-F 2 "" H 3538 3150 50  0000 C CNN
+F 2 "Capacitors_SMD:C_0603" H 3538 3150 50  0001 C CNN
 F 3 "" H 3500 3300 50  0000 C CNN
 	1    3500 3300
@@
 $EndComp
 $Comp
-L ZENER D?
+L ZENER D1
 U 1 1 5775E48B
 P 3500 3900
-F 0 "D?" H 3500 4000 50  0000 C CNN
+F 0 "D1" H 3500 4000 50  0000 C CNN
 F 1 "ZENER" H 3500 3800 50  0000 C CNN
-F 2 "" H 3500 3900 50  0000 C CNN
+F 2 "Diodes_SMD:SOD-123" H 3500 3900 50  0001 C CNN
 F 3 "" H 3500 3900 50  0000 C CNN
 	1    3500 3900
@@
 $EndComp
 $Comp
-L GND #PWR?
+L GND #PWR01
 U 1 1 5775E514
-P 2450 4350
-F 0 "#PWR?" H 2450 4100 50  0001 C CNN
-F 1 "GND" H 2450 4200 50  0000 C CNN
-F 2 "" H 2450 4350 50  0000 C CNN
-F 3 "" H 2450 4350 50  0000 C CNN
-	1    2450 4350
-	1    0    0    -1
-$EndComp
-$Comp
-L VCC #PWR?
+P 2550 4350
+F 0 "#PWR01" H 2550 4100 50  0001 C CNN
+F 1 "GND" H 2550 4200 50  0000 C CNN
+F 2 "" H 2550 4350 50  0000 C CNN
+F 3 "" H 2550 4350 50  0000 C CNN
+	1    2550 4350
+	1    0    0    -1
+$EndComp
+$Comp
+L VCC #PWR02
 U 1 1 5775E532
-P 2450 2650
-F 0 "#PWR?" H 2450 2500 50  0001 C CNN
-F 1 "VCC" H 2450 2800 50  0000 C CNN
-F 2 "" H 2450 2650 50  0000 C CNN
-F 3 "" H 2450 2650 50  0000 C CNN
-	1    2450 2650
-	1    0    0    -1
-$EndComp
-$Comp
-L SW_PUSH SW?
+P 2550 2650
+F 0 "#PWR02" H 2550 2500 50  0001 C CNN
+F 1 "VCC" H 2550 2800 50  0000 C CNN
+F 2 "" H 2550 2650 50  0000 C CNN
+F 3 "" H 2550 2650 50  0000 C CNN
+	1    2550 2650
+	1    0    0    -1
+$EndComp
+$Comp
+L SW_PUSH SW1
 U 1 1 5775E6E6
 P 2700 3850
-F 0 "SW?" H 2850 3960 50  0000 C CNN
+F 0 "SW1" H 2850 3960 50  0000 C CNN
 F 1 "SW_PUSH" H 2700 3770 50  0000 C CNN
-F 2 "" H 2700 3850 50  0000 C CNN
+F 2 "Connect:PINHEAD1-3" H 2700 3850 50  0001 C CNN
 F 3 "" H 2700 3850 50  0000 C CNN
 	1    2700 3850
 	0    -1   -1   0
 $EndComp
-$Comp
-L IRFS7530 Q?
-U 1 1 5775E96F
+Wire Wire Line
+	2550 2650 2550 2800
+Wire Wire Line
+	2350 2800 4450 2800
+Wire Wire Line
+	2700 3500 4150 3500
+Wire Wire Line
+	3100 3350 3100 3650
+Connection ~ 3100 3500
+Wire Wire Line
+	3100 3050 3100 2800
+Connection ~ 3100 2800
+Wire Wire Line
+	2550 4350 2550 4200
+Wire Wire Line
+	2350 4200 6150 4200
+Wire Wire Line
+	3100 3950 3100 4200
+Connection ~ 3100 4200
+Wire Wire Line
+	2700 4150 2700 4200
+Connection ~ 2700 4200
+Wire Wire Line
+	2700 3550 2700 3500
+Wire Wire Line
+	3650 3100 3500 3100
+Wire Wire Line
+	3500 3100 3500 3150
+Wire Wire Line
+	3500 3450 3500 3700
+Connection ~ 3500 3500
+Wire Wire Line
+	3500 4100 3500 4200
+Connection ~ 3500 4200
+Wire Wire Line
+	4050 3500 4050 3750
+Wire Wire Line
+	4050 3750 5550 3750
+Wire Wire Line
+	5550 3750 5550 3500
+Wire Wire Line
+	4850 3500 4850 3750
+Connection ~ 4850 3750
+Wire Wire Line
+	3950 3100 6100 3100
+Wire Wire Line
+	4450 3100 4450 3250
+Wire Wire Line
+	5850 3250 5850 3100
+Connection ~ 5850 3100
+Wire Wire Line
+	5150 3250 5150 3100
+Connection ~ 5150 3100
+Wire Wire Line
+	4450 3650 4450 4200
+Connection ~ 4450 4200
+Wire Wire Line
+	5150 3650 5150 4200
+Connection ~ 5150 4200
+Wire Wire Line
+	5850 4200 5850 3650
+Connection ~ 4050 3500
+Connection ~ 4450 3100
+$Comp
+L CONN_01X02 P7
+U 1 1 577ECAA0
+P 6350 4150
+F 0 "P7" H 6350 4300 50  0000 C CNN
+F 1 "CONN_01X02" V 6450 4150 50  0000 C CNN
+F 2 "Connect:PINHEAD1-2" H 6350 4150 50  0001 C CNN
+F 3 "" H 6350 4150 50  0000 C CNN
+	1    6350 4150
+	1    0    0    -1
+$EndComp
+Connection ~ 5850 4200
+Wire Wire Line
+	6050 4100 6150 4100
+Wire Wire Line
+	6050 3900 6050 4100
+$Comp
+L +12V #PWR03
+U 1 1 577ECC09
+P 6050 3900
+F 0 "#PWR03" H 6050 3750 50  0001 C CNN
+F 1 "+12V" H 6050 4040 50  0000 C CNN
+F 2 "" H 6050 3900 50  0000 C CNN
+F 3 "" H 6050 3900 50  0000 C CNN
+	1    6050 3900
+	1    0    0    -1
+$EndComp
+$Comp
+L Screw_Terminal P3
+U 1 1 577ECE79
+P 4650 2800
+F 0 "P3" H 4650 2900 50  0000 C CNN
+F 1 "Screw_Terminal" H 4450 2700 50  0000 C CNN
+F 2 "sparkparts:M5_Screw_Terminal_12_pin" H 4650 2800 50  0001 C CNN
+F 3 "" H 4650 2800 50  0000 C CNN
+	1    4650 2800
+	1    0    0    -1
+$EndComp
+$Comp
+L Screw_Terminal P4
+U 1 1 577ECEBD
+P 5050 2800
+F 0 "P4" H 5050 2700 50  0000 C CNN
+F 1 "Screw_Terminal" H 4850 2900 50  0000 C CNN
+F 2 "sparkparts:M5_Screw_Terminal_12_pin" H 5050 2800 50  0001 C CNN
+F 3 "" H 5050 2800 50  0000 C CNN
+	1    5050 2800
+	-1   0    0    1
+$EndComp
+Wire Wire Line
+	5250 2800 6100 2800
+Text Notes 3600 2600 0    60   ~ 0
+Fuse holder, 30mm spacing between screw terminals\n
+Text Notes 5550 4550 0    60   ~ 0
+12V supply for optional LED button
+Text Notes 5850 4650 0    60   ~ 0
+12V supplied externally
+Connection ~ 2550 2800
+Connection ~ 2550 4200
+$Comp
+L Pad_Conn P1
+U 1 1 577ED8F0
+P 2150 2800
+F 0 "P1" H 2150 2900 50  0000 C CNN
+F 1 "Pad_Conn" V 2250 2800 50  0000 C CNN
+F 2 "sparkparts:1PAD_6x5mm" H 2150 2800 50  0001 C CNN
+F 3 "" H 2150 2800 50  0000 C CNN
+	1    2150 2800
+	-1   0    0    1
+$EndComp
+$Comp
+L Pad_Conn P2
+U 1 1 577ED942
+P 2150 4200
+F 0 "P2" H 2150 4300 50  0000 C CNN
+F 1 "Pad_Conn" V 2250 4200 50  0000 C CNN
+F 2 "sparkparts:1PAD_6x5mm" H 2150 4200 50  0001 C CNN
+F 3 "" H 2150 4200 50  0000 C CNN
+	1    2150 4200
+	-1   0    0    1
+$EndComp
+$Comp
+L Pad_Conn P6
+U 1 1 577ED99B
+P 6300 3100
+F 0 "P6" H 6300 3200 50  0000 C CNN
+F 1 "Pad_Conn" H 6400 3000 50  0000 C CNN
+F 2 "sparkparts:1PAD_6x5mm" V 6300 3100 50  0001 C CNN
+F 3 "" H 6300 3100 50  0000 C CNN
+	1    6300 3100
+	1    0    0    -1
+$EndComp
+$Comp
+L Pad_Conn P5
+U 1 1 577ED9DE
+P 6300 2800
+F 0 "P5" H 6300 2900 50  0000 C CNN
+F 1 "Pad_Conn" H 6400 2700 50  0000 C CNN
+F 2 "sparkparts:1PAD_6x5mm" H 6300 2800 50  0001 C CNN
+F 3 "" H 6300 2800 50  0000 C CNN
+	1    6300 2800
+	1    0    0    -1
+$EndComp
+$Comp
+L IRFS7530 Q1
+U 1 1 577F004A
 P 4350 3450
-F 0 "Q?" H 4550 3525 50  0000 L CNN
+F 0 "Q1" H 4550 3525 50  0000 L CNN
 F 1 "IRFS7530" H 4550 3450 50  0000 L CNN
 F 2 "sparkparts:D2PAK-7-GDS" H 4550 3375 50  0001 L CIN
@@
 $EndComp
 $Comp
-L IRFS7530 Q?
-U 1 1 5775E99F
+L IRFS7530 Q2
+U 1 1 577F00A7
 P 5050 3450
-F 0 "Q?" H 5250 3525 50  0000 L CNN
+F 0 "Q2" H 5250 3525 50  0000 L CNN
 F 1 "IRFS7530" H 5250 3450 50  0000 L CNN
 F 2 "sparkparts:D2PAK-7-GDS" H 5250 3375 50  0001 L CIN
@@
 $EndComp
 $Comp
-L IRFS7530 Q?
-U 1 1 5775E9D5
+L IRFS7530 Q3
+U 1 1 577F00F2
 P 5750 3450
-F 0 "Q?" H 5950 3525 50  0000 L CNN
+F 0 "Q3" H 5950 3525 50  0000 L CNN
 F 1 "IRFS7530" H 5950 3450 50  0000 L CNN
 F 2 "sparkparts:D2PAK-7-GDS" H 5950 3375 50  0001 L CIN
@@
 	1    0    0    -1
 $EndComp
-Wire Wire Line
-	2450 2650 2450 2800
-Wire Wire Line
-	2450 2800 3100 2800
-Wire Wire Line
-	3100 2800 6100 2800
-Wire Wire Line
-	2700 3500 3100 3500
-Wire Wire Line
-	3100 3500 3500 3500
-Wire Wire Line
-	3500 3500 4050 3500
-Wire Wire Line
-	4050 3500 4150 3500
-Wire Wire Line
-	3100 3350 3100 3500
-Wire Wire Line
-	3100 3500 3100 3650
-Connection ~ 3100 3500
-Wire Wire Line
-	3100 3050 3100 2800
-Connection ~ 3100 2800
-Wire Wire Line
-	2450 4350 2450 4200
-Wire Wire Line
-	2450 4200 2700 4200
-Wire Wire Line
-	2700 4200 3100 4200
-Wire Wire Line
-	3100 4200 3500 4200
-Wire Wire Line
-	3500 4200 4450 4200
-Wire Wire Line
-	4450 4200 5150 4200
-Wire Wire Line
-	5150 4200 5850 4200
-Wire Wire Line
-	3100 3950 3100 4200
-Connection ~ 3100 4200
-Wire Wire Line
-	2700 4150 2700 4200
-Connection ~ 2700 4200
-Wire Wire Line
-	2700 3550 2700 3500
-Wire Wire Line
-	3650 3100 3500 3100
-Wire Wire Line
-	3500 3100 3500 3150
-Wire Wire Line
-	3500 3450 3500 3500
-Wire Wire Line
-	3500 3500 3500 3700
-Connection ~ 3500 3500
-Wire Wire Line
-	3500 4100 3500 4200
-Connection ~ 3500 4200
-Wire Wire Line
-	4050 3500 4050 3750
-Wire Wire Line
-	4050 3750 4850 3750
-Wire Wire Line
-	4850 3750 5550 3750
-Wire Wire Line
-	5550 3750 5550 3500
-Wire Wire Line
-	4850 3500 4850 3750
-Connection ~ 4850 3750
-Wire Wire Line
-	4450 3100 4450 3100
-Wire Wire Line
-	4450 3100 4450 3250
-Wire Wire Line
-	4450 3100 5150 3100
-Wire Wire Line
-	5150 3100 5850 3100
-Wire Wire Line
-	5850 3100 6100 3100
-Wire Wire Line
-	5850 3250 5850 3100
-Connection ~ 5850 3100
-Wire Wire Line
-	5150 3250 5150 3100
-Connection ~ 5150 3100
-Wire Wire Line
-	4450 3650 4450 4200
-Connection ~ 4450 4200
-Wire Wire Line
-	5150 3650 5150 4200
-Connection ~ 5150 4200
-Wire Wire Line
-	5850 4200 5850 3650
-Connection ~ 4050 3500
-Wire Wire Line
-	3950 3100 4450 3100
-Connection ~ 4450 3100
 $EndSCHEMATC
