File: Anti-Spark-Switch.sch (KiCad schematic (older format))
At the start: 16 parts, among them P1 Pad_Conn, P2 Pad_Conn, P3 Screw_Terminal, P4 Screw_Terminal, P5 Pad_Conn, P6 Pad_Conn, P7 CONN_01X02, Q1 IRFS7530, Q2 IRFS7530, Q3 IRFS7530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

Commit message: Rev 1.1 changes
Moved Gate power input from before to after fuse for improved safety
Parts:
- P6: footprint sparkparts:1PAD_6x5mm -> sparkparts:1PAD_8x7mm
Connections:
- wire segments 28 -> 30
Changed lines of the file:
@@
 Connection ~ 4650 3750
-Wire Wire Line
-	4650 3300 4650 3050
-Connection ~ 4650 3050
 Wire Wire Line
 	4100 4600 4100 4450
@@
 F 0 "P6" H 7850 3450 50  0000 C CNN
 F 1 "Pad_Conn" H 7950 3250 50  0000 C CNN
-F 2 "sparkparts:1PAD_6x5mm" V 7850 3350 50  0001 C CNN
+F 2 "sparkparts:1PAD_8x7mm" V 7850 3350 50  0001 C CNN
 F 3 "" H 7850 3350 50  0000 C CNN
 	1    7850 3350
@@
 	1    0    0    -1
 $EndComp
+Wire Wire Line
+	7400 3050 7400 3250
+Wire Wire Line
+	7400 3250 4650 3250
+Wire Wire Line
+	4650 3250 4650 3300
+Connection ~ 7400 3050
 $EndSCHEMATC

Commit message: Text changes to schematic
Other:
- note added: "12V (5V) supplied externally"
- note added: "12V (5V) supply for optional LED button"
- note removed: "12V supplied externally"
- note removed: "12V supply for optional LED button"
Changed lines of the file:
@@
 Fuse holder, 30mm spacing between screw terminals\n
 Text Notes 7100 4800 0    60   ~ 0
-12V supply for optional LED button
+12V (5V) supply for optional LED button
 Text Notes 7400 4900 0    60   ~ 0
-12V supplied externally
+12V (5V) supplied externally
 Connection ~ 4100 3050
 Connection ~ 4100 4450

Commit message: text fixes/passive component footprint changes
Parts:
- C1: footprint Capacitors_SMD:C_0603 -> Capacitors_SMD:C_0603_HandSoldering
- R1, R2, R3: footprint Resistors_SMD:R_0603 -> Resistors_SMD:R_0603_HandSoldering
Changed lines of the file:
@@
 F 0 "R2" V 4730 4050 50  0000 C CNN
 F 1 "1M" V 4650 4050 50  0000 C CNN
-F 2 "Resistors_SMD:R_0603" V 4580 4050 50  0001 C CNN
+F 2 "Resistors_SMD:R_0603_HandSoldering" V 4580 4050 50  0001 C CNN
 F 3 "" H 4650 4050 50  0000 C CNN
 	1    4650 4050
@@
 F 0 "R1" V 4730 3450 50  0000 C CNN
 F 1 "1M" V 4650 3450 50  0000 C CNN
-F 2 "Resistors_SMD:R_0603" V 4580 3450 50  0001 C CNN
+F 2 "Resistors_SMD:R_0603_HandSoldering" V 4580 3450 50  0001 C CNN
 F 3 "" H 4650 3450 50  0000 C CNN
 	1    4650 3450
@@
 F 0 "R3" V 5430 3350 50  0000 C CNN
 F 1 "1K" V 5350 3350 50  0000 C CNN
-F 2 "Resistors_SMD:R_0603" V 5280 3350 50  0001 C CNN
+F 2 "Resistors_SMD:R_0603_HandSoldering" V 5280 3350 50  0001 C CNN
 F 3 "" H 5350 3350 50  0000 C CNN
 	1    5350 3350
@@
 F 0 "C1" H 5075 3650 50  0000 L CNN
 F 1 "1uF" H 5075 3450 50  0000 L CNN
-F 2 "Capacitors_SMD:C_0603" H 5088 3400 50  0001 C CNN
+F 2 "Capacitors_SMD:C_0603_HandSoldering" H 5088 3400 50  0001 C CNN
 F 3 "" H 5050 3550 50  0000 C CNN
 	1    5050 3550

Commit message: Fixed short through LED issue
may still need some tweaking
Connections:
- wire segments 30 -> 32
Changed lines of the file:
@@
 	4100 4600 4100 4450
 Wire Wire Line
-	3900 4450 7700 4450
-Wire Wire Line
-	4650 4200 4650 4450
+	4650 4450 4650 4200
 Connection ~ 4650 4450
 Wire Wire Line
-	4250 4400 4250 4450
+	4250 4450 4250 4400
 Connection ~ 4250 4450
 Wire Wire Line
@@
 Connection ~ 5050 3750
 Wire Wire Line
-	5050 4350 5050 4450
+	5050 4450 5050 4350
 Connection ~ 5050 4450
 Wire Wire Line
@@
 Connection ~ 6700 3350
 Wire Wire Line
-	6000 3900 6000 4450
+	6000 4450 6000 3900
 Connection ~ 6000 4450
 Wire Wire Line
-	6700 3900 6700 4450
+	6700 4450 6700 3900
 Connection ~ 6700 4450
 Wire Wire Line
@@
 	1    0    0    -1
 $EndComp
-Connection ~ 7400 4450
 Wire Wire Line
 	7600 4350 7700 4350
@@
 	4650 3250 4650 3300
 Connection ~ 7400 3050
+Wire Wire Line
+	3900 4450 7400 4450
+Wire Wire Line
+	7500 3350 7500 4450
+Wire Wire Line
+	7500 4450 7700 4450
+Connection ~ 7500 3350
 $EndSCHEMATC

Commit message: updated schematic, changed bom slightly
Parts:
- added R4, R5: 16.5K, Resistors_SMD:R_1206, symbol R
Connections:
- net labels removed: +12V
- wire segments 32 -> 37
Other:
- note added: "LED output"
- note removed: "12V (5V) supplied externally"
- note removed: "12V (5V) supply for optional LED button"
- moved on the sheet: P5, P6, P7
Changed lines of the file:
@@
 LIBS:crf_1
 LIBS:Anti-Spark-Switch-cache
-EELAYER 25 0
+EELAYER 26 0
 EELAYER END
 $Descr A4 11693 8268
@@
 Connection ~ 6400 4000
 Wire Wire Line
-	5500 3350 7650 3350
+	5500 3350 8250 3350
 Wire Wire Line
 	6000 3350 6000 3500
@@
 L CONN_01X02 P7
 U 1 1 577ECAA0
-P 7900 4400
-F 0 "P7" H 7900 4550 50  0000 C CNN
-F 1 "CONN_01X02" V 8000 4400 50  0000 C CNN
-F 2 "Connect:PINHEAD1-2" H 7900 4400 50  0001 C CNN
-F 3 "" H 7900 4400 50  0000 C CNN
-	1    7900 4400
-	1    0    0    -1
-$EndComp
-Wire Wire Line
-	7600 4350 7700 4350
-Wire Wire Line
-	7600 4150 7600 4350
-$Comp
-L +12V #PWR03
-U 1 1 577ECC09
-P 7600 4150
-F 0 "#PWR03" H 7600 4000 50  0001 C CNN
-F 1 "+12V" H 7600 4290 50  0000 C CNN
-F 2 "" H 7600 4150 50  0000 C CNN
-F 3 "" H 7600 4150 50  0000 C CNN
-	1    7600 4150
-	1    0    0    -1
-$EndComp
+P 8400 4400
+F 0 "P7" H 8400 4550 50  0000 C CNN
+F 1 "CONN_01X02" V 8500 4400 50  0000 C CNN
+F 2 "Connect:PINHEAD1-2" H 8400 4400 50  0001 C CNN
+F 3 "" H 8400 4400 50  0000 C CNN
+	1    8400 4400
+	1    0    0    -1
+$EndComp
+Wire Wire Line
+	7800 4350 8200 4350
 $Comp
 L Screw_Terminal P3
@@
 $EndComp
 Wire Wire Line
-	6800 3050 7650 3050
+	6800 3050 8250 3050
 Text Notes 5150 2850 0    60   ~ 0
 Fuse holder, 30mm spacing between screw terminals\n
-Text Notes 7100 4800 0    60   ~ 0
-12V (5V) supply for optional LED button
-Text Notes 7400 4900 0    60   ~ 0
-12V (5V) supplied externally
 Connection ~ 4100 3050
 Connection ~ 4100 4450
@@
 L Pad_Conn P6
 U 1 1 577ED99B
-P 7850 3350
-F 0 "P6" H 7850 3450 50  0000 C CNN
-F 1 "Pad_Conn" H 7950 3250 50  0000 C CNN
-F 2 "sparkparts:1PAD_8x7mm" V 7850 3350 50  0001 C CNN
-F 3 "" H 7850 3350 50  0000 C CNN
-	1    7850 3350
+P 8450 3350
+F 0 "P6" H 8450 3450 50  0000 C CNN
+F 1 "Pad_Conn" H 8550 3250 50  0000 C CNN
+F 2 "sparkparts:1PAD_8x7mm" V 8450 3350 50  0001 C CNN
+F 3 "" H 8450 3350 50  0000 C CNN
+	1    8450 3350
 	1    0    0    -1
 $EndComp
@@
 L Pad_Conn P5
 U 1 1 577ED9DE
-P 7850 3050
-F 0 "P5" H 7850 3150 50  0000 C CNN
-F 1 "Pad_Conn" H 7950 2950 50  0000 C CNN
-F 2 "sparkparts:1PAD_6x5mm" H 7850 3050 50  0001 C CNN
-F 3 "" H 7850 3050 50  0000 C CNN
-	1    7850 3050
+P 8450 3050
+F 0 "P5" H 8450 3150 50  0000 C CNN
+F 1 "Pad_Conn" H 8550 2950 50  0000 C CNN
+F 2 "sparkparts:1PAD_6x5mm" H 8450 3050 50  0001 C CNN
+F 3 "" H 8450 3050 50  0000 C CNN
+	1    8450 3050
 	1    0    0    -1
 $EndComp
@@
 U 1 1 577F004A
 P 5900 3700
-F 0 "Q1" H 6100 3775 50  0000 L CNN
-F 1 "IRFS7530" H 6100 3700 50  0000 L CNN
+F 0 "Q1" H 6100 3850 50  0000 L CNN
+F 1 "IRFS7530" V 6150 3450 50  0000 L CNN
 F 2 "sparkparts:D2PAK-7-GDS" H 6100 3625 50  0001 L CIN
 F 3 "" H 5900 3700 50  0000 L CNN
@@
 U 1 1 577F00A7
 P 6600 3700
-F 0 "Q2" H 6800 3775 50  0000 L CNN
-F 1 "IRFS7530" H 6800 3700 50  0000 L CNN
+F 0 "Q2" H 6800 3850 50  0000 L CNN
+F 1 "IRFS7530" V 6850 3450 50  0000 L CNN
 F 2 "sparkparts:D2PAK-7-GDS" H 6800 3625 50  0001 L CIN
 F 3 "" H 6600 3700 50  0000 L CNN
@@
 U 1 1 577F00F2
 P 7300 3700
-F 0 "Q3" H 7500 3775 50  0000 L CNN
-F 1 "IRFS7530" H 7500 3700 50  0000 L CNN
+F 0 "Q3" H 7550 3850 50  0000 L CNN
+F 1 "IRFS7530" V 7600 3450 50  0000 L CNN
 F 2 "sparkparts:D2PAK-7-GDS" H 7500 3625 50  0001 L CIN
 F 3 "" H 7300 3700 50  0000 L CNN
@@
 	7500 3350 7500 4450
 Wire Wire Line
-	7500 4450 7700 4450
+	7500 4450 8200 4450
 Connection ~ 7500 3350
+$Comp
+L R R4
+U 1 1 5AD7FABD
+P 7800 3650
+F 0 "R4" H 7870 3696 50  0000 L CNN
+F 1 "16.5K" V 7800 3550 43  0000 L CNN
+F 2 "Resistors_SMD:R_1206" V 7730 3650 50  0001 C CNN
+F 3 "" H 7800 3650 50  0001 C CNN
+	1    7800 3650
+	1    0    0    -1
+$EndComp
+$Comp
+L R R5
+U 1 1 5AD7FB17
+P 8050 3650
+F 0 "R5" H 8120 3696 50  0000 L CNN
+F 1 "16.5K" V 8050 3550 43  0000 L CNN
+F 2 "Resistors_SMD:R_1206" V 7980 3650 50  0001 C CNN
+F 3 "" H 8050 3650 50  0001 C CNN
+	1    8050 3650
+	1    0    0    -1
+$EndComp
+Wire Wire Line
+	7800 3050 7800 3500
+Wire Wire Line
+	7800 3450 8050 3450
+Wire Wire Line
+	8050 3450 8050 3500
+Wire Wire Line
+	7800 3800 7800 4350
+Wire Wire Line
+	7800 3850 8050 3850
+Wire Wire Line
+	8050 3850 8050 3800
+Connection ~ 7800 3050
+Connection ~ 7800 3450
+Connection ~ 7800 3850
+Text Notes 7950 4050 0    60   ~ 0
+LED output
 $EndSCHEMATC

Commit message: moved images to new folder, updated a PCB footprint
Parts:
- C1: footprint Capacitors_SMD:C_0603_HandSoldering -> Capacitors_SMD:C_0603
- R1, R2, R3: footprint Resistors_SMD:R_0603_HandSoldering -> Resistors_SMD:R_0603
Changed lines of the file:
@@
 F 0 "R2" V 4730 4050 50  0000 C CNN
 F 1 "1M" V 4650 4050 50  0000 C CNN
-F 2 "Resistors_SMD:R_0603_HandSoldering" V 4580 4050 50  0001 C CNN
+F 2 "Resistors_SMD:R_0603" V 4580 4050 50  0001 C CNN
 F 3 "" H 4650 4050 50  0000 C CNN
 	1    4650 4050
@@
 F 0 "R1" V 4730 3450 50  0000 C CNN
 F 1 "1M" V 4650 3450 50  0000 C CNN
-F 2 "Resistors_SMD:R_0603_HandSoldering" V 4580 3450 50  0001 C CNN
+F 2 "Resistors_SMD:R_0603" V 4580 3450 50  0001 C CNN
 F 3 "" H 4650 3450 50  0000 C CNN
 	1    4650 3450
@@
 F 0 "R3" V 5430 3350 50  0000 C CNN
 F 1 "1K" V 5350 3350 50  0000 C CNN
-F 2 "Resistors_SMD:R_0603_HandSoldering" V 5280 3350 50  0001 C CNN
+F 2 "Resistors_SMD:R_0603" V 5280 3350 50  0001 C CNN
 F 3 "" H 5350 3350 50  0000 C CNN
 	1    5350 3350
@@
 F 0 "C1" H 5075 3650 50  0000 L CNN
 F 1 "1uF" H 5075 3450 50  0000 L CNN
-F 2 "Capacitors_SMD:C_0603_HandSoldering" H 5088 3400 50  0001 C CNN
+F 2 "Capacitors_SMD:C_0603" H 5088 3400 50  0001 C CNN
 F 3 "" H 5050 3550 50  0000 C CNN
 	1    5050 3550

Commit message: schematic changes and updating the netlist
Parts:
- P1, P2, P5: footprint sparkparts:1PAD_6x5mm -> sparkparts:1PAD_8x7mm
Changed lines of the file:
@@
 F 0 "P1" H 3700 3150 50  0000 C CNN
 F 1 "Pad_Conn" V 3800 3050 50  0000 C CNN
-F 2 "sparkparts:1PAD_6x5mm" H 3700 3050 50  0001 C CNN
+F 2 "sparkparts:1PAD_8x7mm" H 3700 3050 50  0001 C CNN
 F 3 "" H 3700 3050 50  0000 C CNN
 	1    3700 3050
@@
 F 0 "P2" H 3700 4550 50  0000 C CNN
 F 1 "Pad_Conn" V 3800 4450 50  0000 C CNN
-F 2 "sparkparts:1PAD_6x5mm" H 3700 4450 50  0001 C CNN
+F 2 "sparkparts:1PAD_8x7mm" H 3700 4450 50  0001 C CNN
 F 3 "" H 3700 4450 50  0000 C CNN
 	1    3700 4450
@@
 F 0 "P5" H 8450 3150 50  0000 C CNN
 F 1 "Pad_Conn" H 8550 2950 50  0000 C CNN
-F 2 "sparkparts:1PAD_6x5mm" H 8450 3050 50  0001 C CNN
+F 2 "sparkparts:1PAD_8x7mm" H 8450 3050 50  0001 C CNN
 F 3 "" H 8450 3050 50  0000 C CNN
 	1    8450 3050

Commit message: changed connector to JST-PH-4 vertical connector, added silkscreen stuff
Parts:
- removed SW1: SW_PUSH, Connect:PINHEAD1-3, symbol SW_PUSH
- D1: footprint Diodes_SMD:SOD-123 -> Diodes_SMD:D_SOD-123F
- P7: value CONN_01X02 -> CONN_01X04; footprint Connect:PINHEAD1-2 -> Connector_JST:JST_PH_B4B-PH-K_1x04_P2.00mm_Vertical; symbol CONN_01X02 -> Conn_01x04
Connections:
- net GND: now also P7.4 (Pin_4)
- net SW_NC: now reaches C1.2, D1.1 (K), Q1.G, Q2.G, Q3.G, R1.2, R2.1
- net SW_NC: now also P7.3 (Pin_3)
- net at P6.1 (P1), Q1.D, Q2.D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: now also P7.1 (Pin_1); no longer P7.2 (P2)
- net at R4.2, R5.2: now also P7.2 (Pin_2); no longer P7.1 (P1)
Other:
- moved on the sheet: R4, R5
Changed lines of the file:
@@
 F 0 "D1" H 5050 4250 50  0000 C CNN
 F 1 "ZENER" H 5050 4050 50  0000 C CNN
-F 2 "Diodes_SMD:SOD-123" H 5050 4150 50  0001 C CNN
+F 2 "Diodes_SMD:D_SOD-123F" H 5050 4150 50  0001 C CNN
 F 3 "" H 5050 4150 50  0000 C CNN
 	1    5050 4150
@@
 $EndComp
 $Comp
-L SW_PUSH SW1
-U 1 1 5775E6E6
-P 4250 4100
-F 0 "SW1" H 4400 4210 50  0000 C CNN
-F 1 "SW_PUSH" H 4250 4020 50  0000 C CNN
-F 2 "Connect:PINHEAD1-3" H 4250 4100 50  0001 C CNN
-F 3 "" H 4250 4100 50  0000 C CNN
-	1    4250 4100
-	0    -1   -1   0
-$EndComp
-Wire Wire Line
-	4100 2900 4100 3050
-Wire Wire Line
-	3900 3050 6000 3050
-Wire Wire Line
-	4250 3750 5700 3750
-Wire Wire Line
-	4650 3600 4650 3900
-Connection ~ 4650 3750
-Wire Wire Line
-	4100 4600 4100 4450
-Wire Wire Line
-	4650 4450 4650 4200
-Connection ~ 4650 4450
-Wire Wire Line
-	4250 4450 4250 4400
-Connection ~ 4250 4450
-Wire Wire Line
-	4250 3800 4250 3750
-Wire Wire Line
-	5200 3350 5050 3350
-Wire Wire Line
-	5050 3350 5050 3400
-Wire Wire Line
-	5050 3700 5050 3950
-Connection ~ 5050 3750
-Wire Wire Line
-	5050 4450 5050 4350
-Connection ~ 5050 4450
-Wire Wire Line
-	5600 3750 5600 4000
-Wire Wire Line
-	5600 4000 7100 4000
-Wire Wire Line
-	7100 4000 7100 3750
-Wire Wire Line
-	6400 3750 6400 4000
-Connection ~ 6400 4000
-Wire Wire Line
-	5500 3350 8250 3350
-Wire Wire Line
-	6000 3350 6000 3500
-Wire Wire Line
-	7400 3500 7400 3350
-Connection ~ 7400 3350
-Wire Wire Line
-	6700 3500 6700 3350
-Connection ~ 6700 3350
-Wire Wire Line
-	6000 4450 6000 3900
-Connection ~ 6000 4450
-Wire Wire Line
-	6700 4450 6700 3900
-Connection ~ 6700 4450
-Wire Wire Line
-	7400 4450 7400 3900
-Connection ~ 5600 3750
-Connection ~ 6000 3350
-$Comp
-L CONN_01X02 P7
+L Conn_01x04 P7
 U 1 1 577ECAA0
-P 8400 4400
-F 0 "P7" H 8400 4550 50  0000 C CNN
-F 1 "CONN_01X02" V 8500 4400 50  0000 C CNN
-F 2 "Connect:PINHEAD1-2" H 8400 4400 50  0001 C CNN
-F 3 "" H 8400 4400 50  0000 C CNN
-	1    8400 4400
-	1    0    0    -1
-$EndComp
-Wire Wire Line
-	7800 4350 8200 4350
+P 8400 4450
+F 0 "P7" H 8400 4600 50  0000 C CNN
+F 1 "CONN_01X04" V 8500 4450 50  0000 C CNN
+F 2 "Connector_JST:JST_PH_B4B-PH-K_1x04_P2.00mm_Vertical" H 8400 4450 50  0001 C CNN
+F 3 "" H 8400 4450 50  0000 C CNN
+	1    8400 4450
+	1    0    0    -1
+$EndComp
 $Comp
 L Screw_Terminal P3
@@
 	-1   0    0    1
 $EndComp
-Wire Wire Line
-	6800 3050 8250 3050
 Text Notes 5150 2850 0    60   ~ 0
 Fuse holder, 30mm spacing between screw terminals\n
-Connection ~ 4100 3050
-Connection ~ 4100 4450
 $Comp
 L Pad_Conn P1
@@
 U 1 1 577F00F2
 P 7300 3700
-F 0 "Q3" H 7550 3850 50  0000 L CNN
-F 1 "IRFS7530" V 7600 3450 50  0000 L CNN
+F 0 "Q3" H 7500 3850 50  0000 L CNN
+F 1 "IRFS7530" V 7525 3450 50  0000 L CNN
 F 2 "sparkparts:D2PAK-7-GDS" H 7500 3625 50  0001 L CIN
 F 3 "" H 7300 3700 50  0000 L CNN
@@
 	1    0    0    -1
 $EndComp
+$Comp
+L R R4
+U 1 1 5AD7FABD
+P 7725 3650
+F 0 "R4" H 7795 3696 50  0000 L CNN
+F 1 "16.5K" V 7725 3550 43  0000 L CNN
+F 2 "Resistors_SMD:R_1206" V 7655 3650 50  0001 C CNN
+F 3 "" H 7725 3650 50  0001 C CNN
+	1    7725 3650
+	1    0    0    -1
+$EndComp
+$Comp
+L R R5
+U 1 1 5AD7FB17
+P 7975 3650
+F 0 "R5" H 8045 3696 50  0000 L CNN
+F 1 "16.5K" V 7975 3550 43  0000 L CNN
+F 2 "Resistors_SMD:R_1206" V 7905 3650 50  0001 C CNN
+F 3 "" H 7975 3650 50  0001 C CNN
+	1    7975 3650
+	1    0    0    -1
+$EndComp
+Text Notes 7825 4400 1    60   ~ 0
+LED output
+Text HLabel 4200 4200 0    60   Input ~ 0
+SW_GND
+Text HLabel 4200 4075 0    60   Input ~ 0
+SW_NC
+Wire Wire Line
+	4100 2900 4100 3050
+Wire Wire Line
+	3900 3050 6000 3050
+Wire Wire Line
+	4250 3750 5700 3750
+Wire Wire Line
+	4650 3600 4650 3900
+Connection ~ 4650 3750
+Wire Wire Line
+	4100 4600 4100 4450
+Wire Wire Line
+	4650 4450 4650 4200
+Connection ~ 4650 4450
+Wire Wire Line
+	4250 4450 4250 4200
+Connection ~ 4250 4450
+Wire Wire Line
+	4250 3750 4250 4075
+Wire Wire Line
+	5200 3350 5050 3350
+Wire Wire Line
+	5050 3350 5050 3400
+Wire Wire Line
+	5050 3700 5050 3950
+Connection ~ 5050 3750
+Wire Wire Line
+	5050 4450 5050 4350
+Connection ~ 5050 4450
+Wire Wire Line
+	5600 3750 5600 4000
+Wire Wire Line
+	5600 4000 7100 4000
+Wire Wire Line
+	7100 4000 7100 3750
+Wire Wire Line
+	6400 3750 6400 4000
+Connection ~ 6400 4000
+Wire Wire Line
+	5500 3350 8250 3350
+Wire Wire Line
+	6000 3350 6000 3500
+Wire Wire Line
+	7400 3500 7400 3350
+Connection ~ 7400 3350
+Wire Wire Line
+	6700 3500 6700 3350
+Connection ~ 6700 3350
+Wire Wire Line
+	6000 4450 6000 3900
+Connection ~ 6000 4450
+Wire Wire Line
+	6700 4450 6700 3900
+Connection ~ 6700 4450
+Wire Wire Line
+	7400 3900 7400 4650
+Connection ~ 5600 3750
+Connection ~ 6000 3350
+Wire Wire Line
+	6800 3050 8250 3050
+Connection ~ 4100 3050
+Connection ~ 4100 4450
 Wire Wire Line
 	7400 3050 7400 3250
@@
 	3900 4450 7400 4450
 Wire Wire Line
-	7500 3350 7500 4450
-Wire Wire Line
-	7500 4450 8200 4450
-Connection ~ 7500 3350
-$Comp
-L R R4
-U 1 1 5AD7FABD
-P 7800 3650
-F 0 "R4" H 7870 3696 50  0000 L CNN
-F 1 "16.5K" V 7800 3550 43  0000 L CNN
-F 2 "Resistors_SMD:R_1206" V 7730 3650 50  0001 C CNN
-F 3 "" H 7800 3650 50  0001 C CNN
-	1    7800 3650
-	1    0    0    -1
-$EndComp
-$Comp
-L R R5
-U 1 1 5AD7FB17
-P 8050 3650
-F 0 "R5" H 8120 3696 50  0000 L CNN
-F 1 "16.5K" V 8050 3550 43  0000 L CNN
-F 2 "Resistors_SMD:R_1206" V 7980 3650 50  0001 C CNN
-F 3 "" H 8050 3650 50  0001 C CNN
-	1    8050 3650
-	1    0    0    -1
-$EndComp
-Wire Wire Line
-	7800 3050 7800 3500
-Wire Wire Line
-	7800 3450 8050 3450
-Wire Wire Line
-	8050 3450 8050 3500
-Wire Wire Line
-	7800 3800 7800 4350
-Wire Wire Line
-	7800 3850 8050 3850
-Wire Wire Line
-	8050 3850 8050 3800
-Connection ~ 7800 3050
-Connection ~ 7800 3450
-Connection ~ 7800 3850
-Text Notes 7950 4050 0    60   ~ 0
-LED output
+	7725 3050 7725 3500
+Wire Wire Line
+	7725 3450 7975 3450
+Wire Wire Line
+	7975 3450 7975 3500
+Wire Wire Line
+	7725 3800 7725 4450
+Wire Wire Line
+	7725 3850 7975 3850
+Wire Wire Line
+	7975 3850 7975 3800
+Connection ~ 7725 3050
+Connection ~ 7725 3450
+Connection ~ 7725 3850
+Wire Wire Line
+	4250 4200 4200 4200
+Wire Wire Line
+	4250 4075 4200 4075
+Wire Wire Line
+	7725 4450 8200 4450
+Wire Wire Line
+	8200 4350 8150 4350
+Wire Wire Line
+	8150 4350 8150 3350
+Connection ~ 8150 3350
+Text HLabel 8050 4550 0    60   Input ~ 0
+SW_NC
+Wire Wire Line
+	8050 4550 8200 4550
+Wire Wire Line
+	7400 4650 8200 4650
+Connection ~ 7400 4450
 $EndSCHEMATC
