File: Anti-Spark-Switch.kicad_pcb (KiCad board)
At the start: 2 copper layers, 16 parts, among them P1 Pad_Conn, P2 Pad_Conn, P3 Screw_Terminal, P4 Screw_Terminal, P5 Pad_Conn, P6 Pad_Conn, P7 CONN_01X02, Q1 IRFS7530, Q2 IRFS7530, Q3 IRFS7530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

Commit message: continued work on PCB
Parts:
- moved R1 8.64 mm to (189.5, 70.9), turned to 270 degrees
- moved R3 6.37 mm to (193.0, 70.9), turned to 90 degrees
- moved D1 5.95 mm to (191.3, 75.4), turned to 180 degrees
- moved C1 4.67 mm to (191.3, 70.9), turned to 270 degrees
- moved P7 3.23 mm to (177.3, 72.5)
- moved SW1 3.23 mm to (177.3, 65.4)
- moved P3 3.15 mm to (197.0, 54.0)
- moved P4 2.97 mm to (227.0, 54.0)
- moved P1 2.52 mm to (177.7, 54.0)
- moved R2 2.30 mm to (187.7, 70.9), turned to 90 degrees
- moved P2 1.70 mm to (176.8, 84.6)
- moved P5 0.41 mm to (243.3, 54.0)
Routing:
- net Net-(C1-Pad2): track 0.00 -> 46.2 mm
- net Net-(P6-Pad1): track 0.00 -> 7.97 mm
- net Net-(C1-Pad1): track 0.00 -> 1.78 mm
Other:
- board outline added: 80 x 43 mm

Commit message: finalized rev 1 PCB, generated gerbers, captured images
Parts:
- moved P6 15.7 mm to (239.0, 85.7)
- moved P2 8.30 mm to (185.0, 85.7)
- moved P1 7.34 mm to (185.0, 53.5)
- moved P7 6.08 mm to (183.4, 72.1)
- moved SW1 6.07 mm to (183.4, 65.3)
- moved P5 4.36 mm to (239.0, 53.5)
Connections:
- SW1 pad 3: (no net) -> +12V
Routing:
- net GND: track 0.00 -> 202.5 mm, vias 0 -> 135
- net Net-(P6-Pad1): track 7.97 -> 104.4 mm, vias 0 -> 133
- net VCC: track 0.00 -> 40.7 mm, vias 0 -> 25
- net Net-(P4-Pad1): track 0.00 -> 26.8 mm, vias 0 -> 25
- net +12V: track 0.00 -> 13.9 mm
- net Net-(C1-Pad2): track 46.2 -> 55.6 mm
- added copper zone on B.Cu, net GND
- added copper zone on F.Cu, net GND
- added copper zone on B.Cu, net Net-(P4-Pad1)
- added copper zone on F.Cu, net Net-(P4-Pad1)
- added copper zone on B.Cu, net Net-(P6-Pad1)
- added copper zone on F.Cu, net Net-(P6-Pad1)
- added copper zone on B.Cu, net VCC
- added copper zone on F.Cu, net VCC
Other:
- board size 80 x 43 mm -> 63.2 x 42 mm
- board text added: "12V SW GND"
- board text added: "GND 12V"
- board text added: "GiS AntiSpark"
- board text added: "IN +"
- board text added: "IN -"
- board text added: "OUT +"
- board text added: "OUT -"
- board text added: "Ver: 1.0 Date: 7/16"
