File: Anti-Spark-Switch.kicad_pcb (KiCad board)
At the start: 2 copper layers, 63.2 x 42 mm, 18 parts, among them P1 Pad_Conn, P2 Pad_Conn, P3 Screw_Terminal, P4 Screw_Terminal, P5 Pad_Conn, P6 Pad_Conn, P7 CONN_01X04, Q1 IRFS7530, Q2 IRFS7530, Q3 IRFS7530

Commit message: improved the PCB a bit
Parts:
- added ?: , Kinetic_Footprints:via-0.45mm, F.Cu at (175.9, 93.4)
- added ?: , Kinetic_Footprints:via-0.45mm, F.Cu at (139.9, 93.4)
- added ?: , Kinetic_Footprints:via-0.45mm, F.Cu at (135.9, 93.4)
- added ?: , Kinetic_Footprints:via-0.45mm, F.Cu at (131.9, 93.4)
- added ?: , Kinetic_Footprints:via-0.45mm, F.Cu at (171.9, 93.4)
- added ?: , Kinetic_Footprints:via-0.45mm, F.Cu at (167.9, 93.4)
- added ?: , Kinetic_Footprints:via-0.45mm, F.Cu at (163.9, 93.4)
- added ?: , Kinetic_Footprints:via-0.45mm, F.Cu at (159.9, 93.4)
- added ?: , Kinetic_Footprints:via-0.45mm, F.Cu at (155.9, 93.4)
- added ?: , Kinetic_Footprints:via-0.45mm, F.Cu at (151.9, 93.4)
- added ?: , Kinetic_Footprints:via-0.45mm, F.Cu at (147.9, 93.4)
- added ?: , Kinetic_Footprints:via-0.45mm, F.Cu at (143.9, 93.4)
- added G***: LOGO, w_logo:Logo_silk_high_voltage_10x8.5mm, F.Cu at (147.3, 82.5)
- moved REF*** 23.1 mm to (170.0, 92.9)
Routing:
- net Net-(P6-Pad1): track 121.9 -> 110.0 mm
Other:
- net class Default: clearance 0.13 -> 0
- rule trace_clearance: 0.13 -> 0
- board text added: "Ver: 1.4 - Fuse MG Date: 5/19/18"
- board text removed: "Ver: 1.4 Date: 5/19/18"

Commit message: PCB has been updated per a fixed screw terminal component
Parts:
- P3, P4: footprint sparkparts:M5_Screw_Terminal_12_pin -> Global_Parts:M5_Screw_Terminal_12_pin
Other:
- net class Default: clearance 0 -> 0.13
- rule trace_clearance: 0 -> 0.13
- board text added: "Ver: 1.5 - Fuse MG Date: 5/27/18"
- board text removed: "Ver: 1.4 - Fuse MG Date: 5/19/18"
Changed lines of the file:
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@@
     (last_trace_width 0.25)
     (user_trace_width 0.5)
-    (trace_clearance 0)
+    (trace_clearance 0.13)
     (zone_clearance 0.254)
     (zone_45_only no)
@@
   (net 7 "Net-(P7-Pad2)")
   (net_class Default "This is the default net class."
-    (clearance 0)
+    (clearance 0.13)
     (trace_width 0.25)
     (via_dia 0.6)
@@
     (add_net "Net-(P7-Pad2)")
     (add_net VCC)
+  )
+  (module Global_Parts:M5_Screw_Terminal_12_pin (layer F.Cu)
+    (at 162.315 82.79)
+    (fp_text reference P4 (at -6.045 -5.1) (layer F.SilkS)
+      (effects (font (size 0.75 0.75) (thickness 0.15)))
+    )
+    (fp_text value Screw_Terminal (at -0.381 6.096) (layer F.Fab)
+      (effects (font (size 0.75 0.75) (thickness 0.15)))
+    )
+    (fp_line (start -5 -5) (end -5 5) (layer F.SilkS) (width 0.05))
+    (fp_line (start -5 5) (end 5 5) (layer F.SilkS) (width 0.05))
+    (fp_line (start 5 5) (end 5 -5) (layer F.SilkS) (width 0.05))
+    (fp_line (start 5 -5) (end -5 -5) (layer F.SilkS) (width 0.05))
+    (fp_circle (center 0 0) (end 1.8 1.8) (layer F.SilkS) (width 0.05))
+    (pad "" np_thru_hole circle (at 0 0) (size 5.3 5.3) (drill 5.3) (layers *.Cu *.Mask))
+    (pad 1 thru_hole circle (at 3.81 -3.81) (size 2.2 2.2) (drill 1.6) (layers *.Cu *.Mask)
+      (net 4 "Net-(P4-Pad1)"))
+    (pad 1 thru_hole circle (at 1.27 -3.81) (size 2.2 2.2) (drill 1.6) (layers *.Cu *.Mask)
+      (net 4 "Net-(P4-Pad1)"))
+    (pad 1 thru_hole circle (at 3.81 -1.27) (size 2.2 2.2) (drill 1.6) (layers *.Cu *.Mask)
+      (net 4 "Net-(P4-Pad1)"))
+    (pad 1 thru_hole circle (at 3.81 1.27) (size 2.2 2.2) (drill 1.6) (layers *.Cu *.Mask)
+      (net 4 "Net-(P4-Pad1)"))
+    (pad 1 thru_hole circle (at 3.81 3.81) (size 2.2 2.2) (drill 1.6) (layers *.Cu *.Mask)
+      (net 4 "Net-(P4-Pad1)"))
+    (pad 1 thru_hole circle (at 1.27 3.81) (size 2.2 2.2) (drill 1.6) (layers *.Cu *.Mask)
+      (net 4 "Net-(P4-Pad1)"))
+    (pad 1 thru_hole circle (at -1.27 3.81) (size 2.2 2.2) (drill 1.6) (layers *.Cu *.Mask)
+      (net 4 "Net-(P4-Pad1)"))
+    (pad 1 thru_hole circle (at -3.81 3.81) (size 2.2 2.2) (drill 1.6) (layers *.Cu *.Mask)
+      (net 4 "Net-(P4-Pad1)"))
+    (pad 1 thru_hole circle (at -3.81 1.27) (size 2.2 2.2) (drill 1.6) (layers *.Cu *.Mask)
+      (net 4 "Net-(P4-Pad1)"))
+    (pad 1 thru_hole circle (at -3.81 -1.27) (size 2.2 2.2) (drill 1.6) (layers *.Cu *.Mask)
+      (net 4 "Net-(P4-Pad1)"))
+    (pad 1 thru_hole circle (at -3.81 -3.81) (size 2.2 2.2) (drill 1.6) (layers *.Cu *.Mask)
+      (net 4 "Net-(P4-Pad1)"))
+    (pad 1 thru_hole circle (at -1.27 -3.81) (size 2.2 2.2) (drill 1.6) (layers *.Cu *.Mask)
+      (net 4 "Net-(P4-Pad1)"))
+  )
+  (module Global_Parts:M5_Screw_Terminal_12_pin (layer F.Cu)
+    (at 132.315 82.79)
+    (fp_text reference P3 (at 5.995 -4.73) (layer F.SilkS)
+      (effects (font (size 0.75 0.75) (thickness 0.15)))
+    )
+    (fp_text value Screw_Terminal (at -0.381 6.096) (layer F.Fab)
+      (effects (font (size 0.75 0.75) (thickness 0.15)))
+    )
+    (fp_line (start -5 -5) (end -5 5) (layer F.SilkS) (width 0.05))
+    (fp_line (start -5 5) (end 5 5) (layer F.SilkS) (width 0.05))
+    (fp_line (start 5 5) (end 5 -5) (layer F.SilkS) (width 0.05))
+    (fp_line (start 5 -5) (end -5 -5) (layer F.SilkS) (width 0.05))
+    (fp_circle (center 0 0) (end 1.8 1.8) (layer F.SilkS) (width 0.05))
+    (pad "" np_thru_hole circle (at 0 0) (size 5.3 5.3) (drill 5.3) (layers *.Cu *.Mask))
+    (pad 1 thru_hole circle (at 3.81 -3.81) (size 2.2 2.2) (drill 1.6) (layers *.Cu *.Mask)
+      (net 1 VCC))
+    (pad 1 thru_hole circle (at 1.27 -3.81) (size 2.2 2.2) (drill 1.6) (layers *.Cu *.Mask)
+      (net 1 VCC))
+    (pad 1 thru_hole circle (at 3.81 -1.27) (size 2.2 2.2) (drill 1.6) (layers *.Cu *.Mask)
+      (net 1 VCC))
+    (pad 1 thru_hole circle (at 3.81 1.27) (size 2.2 2.2) (drill 1.6) (layers *.Cu *.Mask)
+      (net 1 VCC))
+    (pad 1 thru_hole circle (at 3.81 3.81) (size 2.2 2.2) (drill 1.6) (layers *.Cu *.Mask)
+      (net 1 VCC))
+    (pad 1 thru_hole circle (at 1.27 3.81) (size 2.2 2.2) (drill 1.6) (layers *.Cu *.Mask)
+      (net 1 VCC))
+    (pad 1 thru_hole circle (at -1.27 3.81) (size 2.2 2.2) (drill 1.6) (layers *.Cu *.Mask)
+      (net 1 VCC))
+    (pad 1 thru_hole circle (at -3.81 3.81) (size 2.2 2.2) (drill 1.6) (layers *.Cu *.Mask)
+      (net 1 VCC))
+    (pad 1 thru_hole circle (at -3.81 1.27) (size 2.2 2.2) (drill 1.6) (layers *.Cu *.Mask)
+      (net 1 VCC))
+    (pad 1 thru_hole circle (at -3.81 -1.27) (size 2.2 2.2) (drill 1.6) (layers *.Cu *.Mask)
+      (net 1 VCC))
+    (pad 1 thru_hole circle (at -3.81 -3.81) (size 2.2 2.2) (drill 1.6) (layers *.Cu *.Mask)
+      (net 1 VCC))
+    (pad 1 thru_hole circle (at -1.27 -3.81) (size 2.2 2.2) (drill 1.6) (layers *.Cu *.Mask)
+      (net 1 VCC))
   )
   (module w_logo:Logo_silk_high_voltage_10x8.5mm (layer F.Cu)
@@
       (net 1 VCC))
   )
-  (module sparkparts:M5_Screw_Terminal_12_pin (layer F.Cu)
-    (at 132.315 82.79)
-    (fp_text reference P3 (at 5.995 -4.73) (layer F.SilkS)
-      (effects (font (size 0.75 0.75) (thickness 0.15)))
-    )
-    (fp_text value Screw_Terminal (at -0.381 6.096) (layer F.Fab)
-      (effects (font (size 0.75 0.75) (thickness 0.15)))
-    )
-    (fp_line (start -5 -5) (end -5 5) (layer F.SilkS) (width 0.05))
-    (fp_line (start -5 5) (end 5 5) (layer F.SilkS) (width 0.05))
-    (fp_line (start 5 5) (end 5 -5) (layer F.SilkS) (width 0.05))
-    (fp_line (start 5 -5) (end -5 -5) (layer F.SilkS) (width 0.05))
-    (fp_circle (center 0 0) (end 1.8 1.8) (layer F.SilkS) (width 0.05))
-    (pad "" np_thru_hole circle (at 0 0) (size 4.5 4.5) (drill 4.2) (layers *.Cu *.Mask))
-    (pad 1 thru_hole circle (at 3.81 -3.81) (size 2.3 2.3) (drill 1.8) (layers *.Cu *.Mask)
-      (net 1 VCC))
-    (pad 1 thru_hole circle (at 1.27 -3.81) (size 2.3 2.3) (drill 1.8) (layers *.Cu *.Mask)
-      (net 1 VCC))
-    (pad 1 thru_hole circle (at 3.81 -1.27) (size 2.3 2.3) (drill 1.8) (layers *.Cu *.Mask)
-      (net 1 VCC))
-    (pad 1 thru_hole circle (at 3.81 1.27) (size 2.3 2.3) (drill 1.8) (layers *.Cu *.Mask)
-      (net 1 VCC))
-    (pad 1 thru_hole circle (at 3.81 3.81) (size 2.3 2.3) (drill 1.8) (layers *.Cu *.Mask)
-      (net 1 VCC))
-    (pad 1 thru_hole circle (at 1.27 3.81) (size 2.3 2.3) (drill 1.8) (layers *.Cu *.Mask)
-      (net 1 VCC))
-    (pad 1 thru_hole circle (at -1.27 3.81) (size 2.3 2.3) (drill 1.8) (layers *.Cu *.Mask)
-      (net 1 VCC))
-    (pad 1 thru_hole circle (at -3.81 3.81) (size 2.3 2.3) (drill 1.8) (layers *.Cu *.Mask)
-      (net 1 VCC))
-    (pad 1 thru_hole circle (at -3.81 1.27) (size 2.3 2.3) (drill 1.8) (layers *.Cu *.Mask)
-      (net 1 VCC))
-    (pad 1 thru_hole circle (at -3.81 -1.27) (size 2.3 2.3) (drill 1.8) (layers *.Cu *.Mask)
-      (net 1 VCC))
-    (pad 1 thru_hole circle (at -3.81 -3.81) (size 2.3 2.3) (drill 1.8) (layers *.Cu *.Mask)
-      (net 1 VCC))
-    (pad 1 thru_hole circle (at -1.27 -3.81) (size 2.3 2.3) (drill 1.8) (layers *.Cu *.Mask)
-      (net 1 VCC))
-  )
-  (module sparkparts:M5_Screw_Terminal_12_pin (layer F.Cu)
-    (at 162.315 82.79)
-    (fp_text reference P4 (at -6.045 -5.1) (layer F.SilkS)
-      (effects (font (size 0.75 0.75) (thickness 0.15)))
-    )
-    (fp_text value Screw_Terminal (at -0.381 6.096) (layer F.Fab)
-      (effects (font (size 0.75 0.75) (thickness 0.15)))
-    )
-    (fp_line (start -5 -5) (end -5 5) (layer F.SilkS) (width 0.05))
-    (fp_line (start -5 5) (end 5 5) (layer F.SilkS) (width 0.05))
-    (fp_line (start 5 5) (end 5 -5) (layer F.SilkS) (width 0.05))
-    (fp_line (start 5 -5) (end -5 -5) (layer F.SilkS) (width 0.05))
-    (fp_circle (center 0 0) (end 1.8 1.8) (layer F.SilkS) (width 0.05))
-    (pad "" np_thru_hole circle (at 0 0) (size 4.5 4.5) (drill 4.2) (layers *.Cu *.Mask))
-    (pad 1 thru_hole circle (at 3.81 -3.81) (size 2.3 2.3) (drill 1.8) (layers *.Cu *.Mask)
-      (net 4 "Net-(P4-Pad1)"))
-    (pad 1 thru_hole circle (at 1.27 -3.81) (size 2.3 2.3) (drill 1.8) (layers *.Cu *.Mask)
-      (net 4 "Net-(P4-Pad1)"))
-    (pad 1 thru_hole circle (at 3.81 -1.27) (size 2.3 2.3) (drill 1.8) (layers *.Cu *.Mask)
-      (net 4 "Net-(P4-Pad1)"))
-    (pad 1 thru_hole circle (at 3.81 1.27) (size 2.3 2.3) (drill 1.8) (layers *.Cu *.Mask)
-      (net 4 "Net-(P4-Pad1)"))
-    (pad 1 thru_hole circle (at 3.81 3.81) (size 2.3 2.3) (drill 1.8) (layers *.Cu *.Mask)
-      (net 4 "Net-(P4-Pad1)"))
-    (pad 1 thru_hole circle (at 1.27 3.81) (size 2.3 2.3) (drill 1.8) (layers *.Cu *.Mask)
-      (net 4 "Net-(P4-Pad1)"))
-    (pad 1 thru_hole circle (at -1.27 3.81) (size 2.3 2.3) (drill 1.8) (layers *.Cu *.Mask)
-      (net 4 "Net-(P4-Pad1)"))
-    (pad 1 thru_hole circle (at -3.81 3.81) (size 2.3 2.3) (drill 1.8) (layers *.Cu *.Mask)
-      (net 4 "Net-(P4-Pad1)"))
-    (pad 1 thru_hole circle (at -3.81 1.27) (size 2.3 2.3) (drill 1.8) (layers *.Cu *.Mask)
-      (net 4 "Net-(P4-Pad1)"))
-    (pad 1 thru_hole circle (at -3.81 -1.27) (size 2.3 2.3) (drill 1.8) (layers *.Cu *.Mask)
-      (net 4 "Net-(P4-Pad1)"))
-    (pad 1 thru_hole circle (at -3.81 -3.81) (size 2.3 2.3) (drill 1.8) (layers *.Cu *.Mask)
-      (net 4 "Net-(P4-Pad1)"))
-    (pad 1 thru_hole circle (at -1.27 -3.81) (size 2.3 2.3) (drill 1.8) (layers *.Cu *.Mask)
-      (net 4 "Net-(P4-Pad1)"))
-  )
   (module Capacitors_SMD:C_0603 (layer F.Cu)
     (at 124.574 99.477 180)
@@
     (effects (font (size 0.75 0.75) (thickness 0.1875)))
   )
-  (gr_text "Ver: 1.4 - Fuse\nMG Date: 5/19/18" (at 176.15 100.545 90) (layer F.SilkS)
+  (gr_text "Ver: 1.5 - Fuse\nMG Date: 5/27/18" (at 176.15 100.545 90) (layer F.SilkS)
     (effects (font (size 1 1) (thickness 0.25)))
   )
